Commit message: Resolved visual anomalies with system. URDF now visually complete & controllable with joint states. Pose manipulation for movement incoming.

File: ros_package/wallbot_urdf/urdf/wallbot.urdf (robot description, URDF)
Before this commit: robot wallbot, 13 links, 12 joints
Joints:
- joint base_to_bottom_left_socket: origin xyz=0.4 0 -0.5 -> xyz=0.4 0 -0.3
- joint base_to_bottom_right_socket: origin xyz=-0.4 0 -0.5 -> xyz=-0.4 0 -0.3
- joint base_to_top_left_socket: origin xyz=0.4 0 0.5 -> xyz=0.4 0 0.3
- joint base_to_top_right_socket: origin xyz=-0.4 0 0.5 -> xyz=-0.4 0 0.3
- joint bottom_left_prismatic_joint: axis 1 0 0 -> 0 0 1; origin xyz=0 0 1 -> xyz=0 0 2
- joint bottom_left_socket_cable_connector: origin xyz=0 1 0 -> xyz=0 0 0 rpy=0 2.24159 0
- joint bottom_right_prismatic_joint: axis 1 0 0 -> 0 0 1; origin xyz=0 0 1 -> xyz=0 0 2
- joint bottom_right_socket_cable_connector: origin xyz=0 1 0 -> xyz=0 0 0 rpy=0 -2.24159 0
- joint top_left_prismatic_joint: axis 1 0 0 -> 0 0 1; origin xyz=0 0 1 -> xyz=0 0 2
- joint top_left_socket_cable_connector: origin xyz=0 1 0 -> xyz=0 0 0 rpy=0 0.9 0
- joint top_right_prismatic_joint: axis 1 0 0 -> 0 0 1; origin xyz=0 0 1 -> xyz=0 0 2
- joint top_right_socket_cable_connector: origin xyz=0 0 0 -> xyz=0 0 0 rpy=0 -0.9 0
