Commit message: Joint Trajectory controller enabled in gazebo classic. Bugs with simulation to be fixed )(collision/gravity)

File: ros_package/wallbot_tl_root/urdf/wallbot.urdf (robot description, URDF)
Before this commit: robot wallbot, 14 links, 13 joints
Links:
- link bottom_left_anchor: mass None -> 0.1; geometry collision box size=0.01 0.01 0.01; visual cylinder length=0.4 radius=0.1
- link bottom_left_cable: mass None -> 0.1; geometry collision box size=0.01 0.01 0.01; visual cylinder length=4 radius=0.01
- link bottom_left_socket: mass None -> 0.1; geometry collision box size=0.01 0.01 0.01; visual sphere radius=0.075
- link bottom_right_anchor: mass None -> 0.1; geometry collision box size=0.01 0.01 0.01; visual cylinder length=0.4 radius=0.1
- link bottom_right_cable: mass None -> 0.1; geometry collision box size=0.01 0.01 0.01; visual cylinder length=4 radius=0.01
- link bottom_right_socket: mass None -> 0.1; geometry collision box size=0.01 0.01 0.01; visual sphere radius=0.075
- link central_body: mass None -> 0.1; geometry collision box size=0.01 0.01 0.01; visual box size=0.8 0.5 0.6
- link tl_anchor: mass None -> 0.1; geometry collision box size=0.01 0.01 0.01
- link top_left_anchor: mass None -> 0.1; geometry collision box size=0.01 0.01 0.01; visual cylinder length=0.4 radius=0.1
- link top_left_cable: mass None -> 0.1; geometry collision box size=0.01 0.01 0.01; visual cylinder length=4 radius=0.01
- link top_left_socket: mass None -> 0.1; geometry collision box size=0.01 0.01 0.01; visual sphere radius=0.075
- link top_right_anchor: mass None -> 0.1; geometry collision box size=0.01 0.01 0.01; visual cylinder length=0.4 radius=0.1
- link top_right_cable: mass None -> 0.1; geometry collision box size=0.01 0.01 0.01; visual cylinder length=4 radius=0.01
- link top_right_socket: mass None -> 0.1; geometry collision box size=0.01 0.01 0.01; visual sphere radius=0.075

Commit message: Wallbot body updated to use stl mesh design

File: ros_package/wallbot_tl_root/urdf/wallbot.urdf (robot description, URDF)
Before this commit: robot wallbot, 14 links, 13 joints
Links:
- link central_body: geometry collision box size=0.01 0.01 0.01; visual mesh filename=model://wallbot_body.stl scale=0.002 0.002 0.002

Commit message: gui and gazebo launch with single command

File: ros_package/wallbot_tl_root/urdf/wallbot.urdf (robot description, URDF)
Before this commit: robot wallbot, 14 links, 13 joints
Links:
- added link front_ndvi_link, mass 0.05; visual box size=0.04 0.04 0.02
- added link front_ndvi_optical_frame, mass 1e-6
- added link front_rgb_link, mass 0.05; visual box size=0.04 0.04 0.02
- added link front_rgb_optical_frame, mass 1e-6
Joints:
- added joint front_ndvi_joint: type fixed, parent central_body, child front_ndvi_link, origin xyz=0.22 0.06 0.30 rpy=0 0 0
- added joint front_ndvi_optical_joint: type fixed, parent front_ndvi_link, child front_ndvi_optical_frame, origin xyz=0 0 0 rpy=-1.57079632679 0 -1.57079632679
- added joint front_rgb_joint: type fixed, parent central_body, child front_rgb_link, origin xyz=0.20 0.00 0.30 rpy=0 0 0
- added joint front_rgb_optical_joint: type fixed, parent front_rgb_link, child front_rgb_optical_frame, origin xyz=0 0 0 rpy=-1.57079632679 0 -1.57079632679
